Commit message: Moslty accurate urdf (apart from the link to the Senze3D)

File: zoidstein_description/urdf/zoidstein_camera.urdf.xacro (robot description, xacro)
@@ -1,34 +1,61 @@
 <?xml version="1.0"?>
+<!-- Source: https://github.com/corot/thorp/blob/master/thorp_bringup/urdf/thorp.urdf.xacro#L112 -->
 <robot xmlns:xacro="http://www.ros.org/wiki/xacro">
-    <xacro:macro name="zoidstein_camera">
-        <link name="camera_link"/>
-        <link name="camera_depth_frame"/>
-        <link name="camera_rgb_frame"/>
-        <link name="camera_rgb_optical_frame"/>
-        <link name="camera_depth_optical_frame"/>
-        <joint name="camera_joint" type="fixed">
-            <origin xyz="" rpy="" />
-            <parent link="" />
-            <child link="camera_link" />
+    <xacro:macro name="zoidstein_camera"
+                 params="camera_parent camera_origin_x camera_origin_y camera_origin_z camera_origin_roll camera_origin_pitch camera_origin_yaw">
+        <link name="senz3d_rgb_frame"/>
+        <link name="senz3d_rgb_optical_frame"/>
+        <link name="senz3d_depth_frame"/>
+        <link name="senz3d_depth_optical_frame"/>
+        <joint name="senz3d_camera_joint" type="fixed">
+            <!-- <origin xyz="-0.045 -0.062 0.345" rpy="${M_PI/2 + 0.907571211037} 0.0 ${M_PI/2}"/> -->
+            <origin xyz="${camera_origin_x} ${camera_origin_y} ${camera_origin_z}"
+                    rpy="${camera_origin_roll} ${camera_origin_pitch} ${camera_origin_yaw}"/>
+            <parent link="${camera_parent}"/>
+            <child link="senz3d_camera_link"/>
         </joint>
-        <joint name="camera_depth_joint" type="fixed">
-            <origin xyz="0 0.018 0" rpy="0 0 0" />
-            <parent link="camera_link" />
-            <child link="camera_depth_frame" />
+        <link name="senz3d_camera_link">
+            <visual>
+                <origin xyz="0.0 0.0 0.0" rpy="0.0 0.0 0.0"/>
+                <geometry>
+                    <!-- As we don't have a Senz3D mesh, use a deformed Asus Xtion Pro instead -->
+                    <mesh filename="package://turtlebot_description/meshes/sensors/asus_xtion_pro_live.dae"
+                          scale="0.0006 0.0015 0.001"/>
+                </geometry>
+            </visual>
+            <collision>
+                <origin xyz="0.0 0.0 -0.005" rpy="0 0 0"/>
+                <geometry>
+                    <box size="0.11 0.04 0.04"/>
+                </geometry>
+            </collision>
+            <inertial>
+                <mass value="0.271"/>
+                <origin xyz="0 0 0"/>
+                <inertia ixx="0.001" ixy="0.0" ixz="0.0"
+                         iyy="0.001" iyz="0.0"
+                         izz="0.001"/>
+            </inertial>
+        </link>
+        <!-- Add frames for RGB and depth optical axes -->
+        <joint name="senz3d_rgb_joint" type="fixed">
+            <origin xyz="0.0125 0.0 0.0" rpy="0.0 0.0 0.0"/>
+            <parent link="senz3d_camera_link"/>
+            <child link="senz3d_rgb_frame"/>
         </joint>
-        <joint name="camera_depth_optical_joint" type="fixed">
-            <origin xyz="0 0 0" rpy="${-M_PI/2} 0 ${-M_PI/2}" />
-            <parent link="camera_depth_frame" />
-            <child link="camera_depth_optical_frame" />
+        <joint name="senz3d_rgb_optical_joint" type="fixed">
+            <origin xyz="0.0 0.0 0.0" rpy="0.0 0.0 ${M_PI}"/>
+            <parent link="senz3d_rgb_frame"/>
+            <child link="senz3d_rgb_optical_frame"/>
         </joint>
-        <joint name="camera_rgb_joint" type="fixed">
-            <origin xyz="0 -0.005 0" rpy="0 0 0" />
-            <parent link="camera_link" />
-            <child link="camera_rgb_frame" />
+        <joint name="senz3d_depth_joint" type="fixed">
+            <origin xyz="-0.0125 0.0 0.0" rpy="0.0 0.0 0.0"/>
+            <parent link="senz3d_camera_link"/>
+            <child link="senz3d_depth_frame"/>
         </joint>
-        <joint name="camera_rgb_optical_joint" type="fixed">
-            <origin xyz="0 0 0" rpy="${-M_PI/2} 0 ${-M_PI/2}" />
-            <parent link="camera_rgb_frame" />
-            <child link="camera_rgb_optical_frame" />
+        <joint name="senz3d_depth_optical_joint" type="fixed">
+            <origin xyz="0.0 0.0 0.0" rpy="0.0 0.0 ${M_PI}"/>
+            <parent link="senz3d_depth_frame"/>
+            <child link="senz3d_depth_optical_frame"/>
         </joint>
     </xacro:macro>

File: zoidstein_description/urdf/zoidstein_head.urdf.xacro (robot description, xacro)
@@ -7,26 +7,26 @@
         <link name="gaze" />
         <joint name="base_joint" type="fixed">
+            <parent link="base_link"/>
             <child link="neck_yaw_link"/>
-            <parent link="base_link"/>
             <origin xyz="0 0 0" rpy="0 0 0" />
         </joint>
-        <joint name="neck_yaw" type="revolute">
+        <joint name="neck_yaw_joint" type="revolute">
             <parent link="base_link"/>
             <child link="neck_yaw_link"/>
-            <origin xyz="0.1 0 0" rpy="0 -1.57 0"/>
-            <axis xyz="1 0 0"/>
-            <limit velocity="1.0" effort="30" lower="-1.0" upper="1.0" />
+            <origin xyz="0 0 0.0545" rpy="0 0 0"/>
+            <axis xyz="0 0 1"/>
+            <limit velocity="1.0" effort="1" lower="-0.8726" upper="0.8726" />
         </joint>
-        <joint name="neck_pitch" type="revolute">
-            <parent link="neck_roll_link"/>
+        <joint name="neck_pitch_joint" type="revolute">
+            <parent link="neck_yaw_link"/>
             <child link="neck_pitch_link"/>
-            <origin xyz="0.1 0 0" rpy="-1.57 0 0"/>
+            <origin xyz="0 0 0.02867" rpy="0 0 0"/>
             <axis xyz="0 1 0"/>
-            <limit velocity="0.78" effort="30" lower="-0.8" upper="0.8" />
+            <limit velocity="1.0" effort="1" lower="-0.8726" upper="0.8726" />
         </joint>
         <joint name="gaze_joint" type="fixed">
             <parent link="neck_pitch_link"/>
             <child link="gaze"/>
-            <origin xyz="0.05 0 -0.1" rpy="0 1.57 0"/>
+            <origin xyz="0.0556 0 0.06578" rpy="0 0 0"/>
         </joint>
     </xacro:macro>

File: zoidstein_description/urdf/zoidstein_robot.urdf.xacro (robot description, xacro)
@@ -1,10 +1,12 @@
 <?xml version="1.0"?>
 <robot xmlns:xacro="http://ros.org/wiki/xacro" name="zoidstein">
-    <xacro:include filename="$(find zoidstein_description)/urdf/zoidstein_head.urdf.xacro" />
-    <xacro:include filename="$(find zoidstein_description)/urdf/zoidstein_camera.urdf.xacro" />
+    <xacro:include filename="$(find zoidstein_description)/urdf/zoidstein_head.urdf.xacro"/>
+    <xacro:include filename="$(find zoidstein_description)/urdf/zoidstein_camera.urdf.xacro"/>
     <!-- Properties -->
-    <xacro:property name="pi" value="3.14159265359" />
+    <xacro:property name="pi" value="3.14159265359"/>
+    <xacro:property name="M_PI" value="3.14159265359"/>
     <!-- Head and camera -->
     <xacro:zoidstein_head/>
-    <xacro:zoidstein_camera/>
+    <xacro:zoidstein_camera camera_parent="base_link" camera_origin_x="0.5" camera_origin_y="0" camera_origin_z="0"
+                            camera_origin_roll="0" camera_origin_pitch="0" camera_origin_yaw="0"/>
 </robot>
