Commit message: Senz3d moves based on distance to sensor

File: zoidstein_description/urdf/senz3d.urdf.xacro (robot description, xacro)
@@ -2,5 +2,5 @@
 <!-- Source: https://github.com/corot/thorp/blob/master/thorp_bringup/urdf/thorp.urdf.xacro#L112 -->
 <robot xmlns:xacro="http://www.ros.org/wiki/xacro">
-    <xacro:macro name="zoidstein_camera"
+    <xacro:macro name="senz3d"
                  params="camera_parent camera_origin_x camera_origin_y camera_origin_z camera_origin_roll camera_origin_pitch camera_origin_yaw">
         <link name="senz3d_rgb_frame"/>

File: zoidstein_description/urdf/zoidstein_robot.urdf.xacro (robot description, xacro)
@@ -2,5 +2,6 @@
 <robot xmlns:xacro="http://ros.org/wiki/xacro" name="zoidstein">
     <xacro:include filename="$(find zoidstein_description)/urdf/zoidstein_head.urdf.xacro"/>
-    <xacro:include filename="$(find zoidstein_description)/urdf/zoidstein_camera.urdf.xacro"/>
+    <xacro:include filename="$(find zoidstein_description)/urdf/zoidstein_camera_joint.urdf.xacro"/>
+    <xacro:include filename="$(find zoidstein_description)/urdf/senz3d.urdf.xacro"/>
     <!-- Properties -->
     <xacro:property name="pi" value="3.14159265359"/>
@@ -8,5 +9,6 @@
     <!-- Head and camera -->
     <xacro:zoidstein_head/>
-    <xacro:zoidstein_camera camera_parent="base_link" camera_origin_x="0.5" camera_origin_y="0" camera_origin_z="0"
+    <xacro:zoidstein_camera_joint/>
+    <xacro:senz3d camera_parent="camera_link" camera_origin_x="0.01682" camera_origin_y="-0.03898" camera_origin_z="0"
                             camera_origin_roll="0" camera_origin_pitch="0" camera_origin_yaw="0"/>
 </robot>
